File: PCB_inzynierka/schemat_ideowy/Matryca_LED.kicad_sch (KiCad schematic)
At the start: 129 parts

Commit message: obie plytki pcb przygotowane, schematy ideowe opisane
Other:
- company: (none) -> AGH
- title: (none) -> Matryca 8x8 Led argb
Changed lines of the file:
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@@
 	(generator_version "9.0")
 	(paper "A3" portrait)
+	(title_block
+		(title "Matryca 8x8 Led argb")
+		(date "2025-11-12")
+		(rev "1")
+		(company "AGH")
+		(comment 1 "Autor: Krystian Bajerski")
+		(comment 2 "Promotor: dr inż. Agnieszka Dąbrowska-Boruch")
+	)
 	(junction
 		(at 133.35 151.13)
