File: PCB_inzynierka/schemat_ideowy/Mul_Mux_Reed_Switches.kicad_sch (KiCad schematic)
At the start: 80 parts, among them SW10 SW_Reed, SW11 SW_Reed, SW12 SW_Reed, SW13 SW_Reed, SW14 SW_Reed, SW15 SW_Reed, SW16 SW_Reed, SW17 SW_Reed, SW18 SW_Reed, SW19 SW_Reed, SW20 SW_Reed, SW21 SW_Reed, SW22 SW_Reed, SW23 SW_Reed, SW24 SW_Reed, SW25 SW_Reed, SW26 SW_Reed, SW27 SW_Reed, SW28 SW_Reed, SW29 SW_Reed, SW30 SW_Reed, SW31 SW_Reed, SW32 SW_Reed, SW33 SW_Reed, SW34 SW_Reed, SW35 SW_Reed, SW36 SW_Reed, SW37 SW_Reed, SW38 SW_Reed, SW39 SW_Reed, SW40 SW_Reed, SW41 SW_Reed, SW42 SW_Reed, SW43 SW_Reed, SW44 SW_Reed, SW45 SW_Reed, SW46 SW_Reed, SW47 SW_Reed, SW48 SW_Reed, SW49 SW_Reed, SW50 SW_Reed, SW51 SW_Reed, SW52 SW_Reed, SW53 SW_Reed, SW54 SW_Reed, SW55 SW_Reed, SW56 SW_Reed, SW57 SW_Reed, SW58 SW_Reed, SW59 SW_Reed, SW60 SW_Reed, SW61 SW_Reed, SW62 SW_Reed, SW63 SW_Reed, SW64 SW_Reed, SW65 SW_Reed, SW66 SW_Reed, SW67 SW_Reed, SW68 SW_Reed, SW69 SW_Reed, SW70 SW_Reed, SW71 SW_Reed, SW72 SW_Reed, SW9 SW_Reed, U2 74HC4051D_653, U3 74HC4051D_653, U4 74HC4051D_653, U5 74HC4051D_653, U6 74HC4051D_653, U7 74HC4051D_653, U8 74HC4051D_653, U9 74HC4051D_653

Commit message: obie plytki pcb przygotowane, schematy ideowe opisane
Other:
- company: (none) -> AGH
- title: (none) -> Detekcja pionków - demultipleksery i kontaktrony
Changed lines of the file:
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@@
 	(generator_version "9.0")
 	(paper "A4")
+	(title_block
+		(title "Detekcja pionków - demultipleksery i kontaktrony")
+		(date "2025-11-12")
+		(rev "1")
+		(company "AGH")
+		(comment 1 "Autor: Krystian Bajerski")
+		(comment 2 "Promotor: dr inż. Agnieszka Dąbrowska-Boruch")
+	)
 	(junction
 		(at 210.82 110.49)
